Commit message: Tune start position of robot in simulation

File: catkin_workspace/src/applications/ropod_demo_dec_2017/config/shape/floorplan_ropod_demo.urdf (robot description, URDF)
Before this commit: robot Floorplan_demo_ROPOD, 1 links, 0 joints
Links:
- link map: geometry collision mesh filename=package://ropod_demo_dec_2017/config/shape/heightmap_sim.stl scale=0.0015 0.0015 0.002; visual mesh filename=package://ropod_demo_dec_2017/config/shape/heightmap_sim.stl scale=0.0015 0.0015 0.002
