Commit message: Remove ROPOD specific packages and remove dependency of ED to ROPOD packages

File: catkin_workspace/src/functionalities/ED/ed_object_models/models/hospital_test/walls/shape/floorplan_ropod_demo.urdf (robot description, URDF)
Before this commit: robot Floorplan_demo_ROPOD, 1 links, 0 joints
Links:
- link map: geometry collision mesh filename=package://pico_navigation_test/config/shape/heightmap_sim.s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 scale=0.0015 0.0015 0.002; visual mesh filename=package://pico_navigation_test/config/shape/heightmap_sim.s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 scale=0.0015 0.0015 0.002
